Commit message: update

File: urdf_fix_inertial/urdf/R5a.urdf (robot description, URDF)
Before this commit: robot R5a, 9 links, 8 joints
Joints:
- joint ${prefix}_arm_joint1: child link1 -> ${prefix}_arm_link1; parent base_link -> ${prefix}_arm_base_link
- joint ${prefix}_arm_joint2: child link2 -> ${prefix}_arm_link2; parent link1 -> ${prefix}_arm_link1
- joint ${prefix}_arm_joint3: child link3 -> ${prefix}_arm_link3; parent link2 -> ${prefix}_arm_link2
- joint ${prefix}_arm_joint4: child link4 -> ${prefix}_arm_link4; parent link3 -> ${prefix}_arm_link3
- joint ${prefix}_arm_joint5: child link5 -> ${prefix}_arm_link5; parent link4 -> ${prefix}_arm_link4
- joint ${prefix}_arm_joint6: child link6 -> ${prefix}_arm_link6; parent link5 -> ${prefix}_arm_link5
- joint ${prefix}_arm_joint7: child link7 -> ${prefix}_arm_link7; parent link6 -> ${prefix}_arm_link6
- joint ${prefix}_arm_joint8: child link8 -> ${prefix}_arm_link8; parent link6 -> ${prefix}_arm_link6
